File: Controller_extLED_withDiagnosis/Controller_extLED_PROFETwithDiagnosis.kicad_pcb (KiCad board)
At the start: 2 copper layers, 75 x 60 mm, 17 parts, among them J1 BAT, J2 Switch, J3 RJ12, J4 RJ12, U1 Arduino_Nano_v3.x, U2 BTS

Commit message: updated logo and silkscreen
Other:
- board text added: "BTSXXX w/ Diagnosis Version 2022_12"

Commit message: DRC weirness
Routing:
- net /RX: track 111.4 -> 109.9 mm
- net /TX: track 76.7 -> 75.3 mm
Changed lines of the file:
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@@
       (drillshape 0)
       (scaleselection 1)
-      (outputdirectory "")
+      (outputdirectory "gerber/")
     )
   )
@@
   (net 35 "Net-(U1-Pad5)")
   (footprint "Connector_RJ:RJ12_Amphenol_54601" (layer "F.Cu")
-    (at 97.57 103.83 -90)
+    (at 97.54 103.79 -90)
     (descr "RJ12 connector  https://cdn.amphenol-icc.com/media/wysiwyg/files/drawing/c-bmj-0082.pdf")
     (tags "RJ12 connector")
@@
     (property "Sheetname" "")
     (attr through_hole)
-    (fp_text reference "U1" (at 7.62 5.08 90) (layer "B.SilkS")
+    (fp_text reference "U1" (at 7.62 1.85 90) (layer "B.SilkS")
       (effects (font (size 1 1) (thickness 0.15)) (justify mirror))
     )
@@
   (segment (start 93.8 94.4) (end 93.2 95) (width 0.25) (layer "F.Cu") (net 8))
   (segment (start 151.4 85.8) (end 153.4 87.8) (width 0.8) (layer "F.Cu") (net 9))
-  (segment (start 95.03 107.64) (end 92 104.61) (width 0.8) (layer "F.Cu") (net 9))
-  (segment (start 92 94.995198) (end 92 96.2) (width 0.8) (layer "F.Cu") (net 9))
+  (segment (start 92 104.61) (end 95.03 107.64) (width 0.8) (layer "F.Cu") (net 9))
   (segment (start 148.4 105.6) (end 147.61 104.81) (width 0.8) (layer "F.Cu") (net 9))
-  (segment (start 95.03 93.04) (end 93.955198 93.04) (width 0.8) (layer "F.Cu") (net 9))
   (segment (start 96.2 85.8) (end 151.4 85.8) (width 0.8) (layer "F.Cu") (net 9))
-  (segment (start 153.4 104.4) (end 152.2 105.6) (width 0.8) (layer "F.Cu") (net 9))
-  (segment (start 95.03 107.64) (end 95.03 107.903731) (width 0.25) (layer "F.Cu") (net 9))
+  (segment (start 93.955198 93.04) (end 92 94.995198) (width 0.8) (layer "F.Cu") (net 9))
   (segment (start 147.61 104.81) (end 147.61 103.31) (width 0.8) (layer "F.Cu") (net 9))
   (segment (start 95.03 93.04) (end 93 91.01) (width 0.8) (layer "F.Cu") (net 9))
-  (segment (start 92 104.61) (end 92 94.995198) (width 0.8) (layer "F.Cu") (net 9))
-  (segment (start 93 91.01) (end 93 89) (width 0.8) (layer "F.Cu") (net 9))
   (segment (start 153.4 87.8) (end 153.4 104.4) (width 0.8) (layer "F.Cu") (net 9))
+  (segment (start 95.03 93.04) (end 93.955198 93.04) (width 0.8) (layer "F.Cu") (net 9))
+  (segment (start 153.4 104.4) (end 152.2 105.6) (width 0.8) (layer "F.Cu") (net 9))
+  (segment (start 93 91.01) (end 93 89) (width 0.8) (layer "F.Cu") (net 9))
+  (segment (start 92 94.995198) (end 92 104.61) (width 0.8) (layer "F.Cu") (net 9))
   (segment (start 152.2 105.6) (end 148.4 105.6) (width 0.8) (layer "F.Cu") (net 9))
   (segment (start 93 89) (end 96.2 85.8) (width 0.8) (layer "F.Cu") (net 9))
-  (segment (start 93.955198 93.04) (end 92 94.995198) (width 0.8) (layer "F.Cu") (net 9))
-  (segment (start 97.57 108.91) (end 99 107.48) (width 0.25) (layer "F.Cu") (net 10))
-  (segment (start 97.57 95.57) (end 97.57 96.23) (width 0.25) (layer "F.Cu") (net 10))
   (segment (start 97.57 108.91) (end 98.89 108.91) (width 0.8) (layer "F.Cu") (net 10))
   (segment (start 146.84 100) (end 150.15 103.31) (width 0.8) (layer "F.Cu") (net 10))
-  (segment (start 97.57 94.31) (end 97.57 95.57) (width 0.25) (layer "F.Cu") (net 10))
+  (segment (start 96.2 104.6) (end 96.8 105.2) (width 0.25) (layer "F.Cu") (net 10))
+  (segment (start 96.8 105.2) (end 98 105.2) (width 0.25) (layer "F.Cu") (net 10))
+  (segment (start 98 105.2) (end 99 106.2) (width 0.25) (layer "F.Cu") (net 10))
+  (segment (start 97.57 100.03) (end 96.2 101.4) (width 0.25) (layer "F.Cu") (net 10))
   (segment (start 107.8 100) (end 146.84 100) (width 0.8) (layer "F.Cu") (net 10))
-  (segment (start 98 105.2) (end 96.8 105.2) (width 0.25) (layer "F.Cu") (net 10))
-  (segment (start 96.2 104.6) (end 96.2 101.4) (width 0.25) (layer "F.Cu") (net 10))
-  (segment (start 99 106.2) (end 98 105.2) (width 0.25) (layer "F.Cu") (net 10))
-  (segment (start 96.8 105.2) (end 96.2 104.6) (width 0.25) (layer "F.Cu") (net 10))
   (segment (start 98.89 108.91) (end 107.8 100) (width 0.8) (layer "F.Cu") (net 10))
-  (segment (start 99 107.48) (end 99 106.2) (width 0.25) (layer "F.Cu") (net 10))
-  (segment (start 97.57 108.17) (end 97.57 108.91) (width 0.25) (layer "F.Cu") (net 10))
-  (segment (start 97.57 100.03) (end 97.57 95.57) (width 0.25) (layer "F.Cu") (net 10))
-  (segment (start 96.2 101.4) (end 97.57 100.03) (width 0.25) (layer "F.Cu") (net 10))
+  (segment (start 99 106.2) (end 99 107.48) (width 0.25) (layer "F.Cu") (net 10))
+  (segment (start 97.57 94.31) (end 97.57 100.03) (width 0.25) (layer "F.Cu") (net 10))
+  (segment (start 96.2 101.4) (end 96.2 104.6) (width 0.25) (layer "F.Cu") (net 10))
+  (segment (start 99 107.48) (end 97.57 108.91) (width 0.25) (layer "F.Cu") (net 10))
   (segment (start 135 112.8) (end 135 111.6) (width 0.8) (layer "F.Cu") (net 11))
   (segment (start 130.59952 117.20048) (end 135 112.8) (width 0.8) (layer "F.Cu") (net 11))
